File: cutoff/cutoff.kicad_pcb (KiCad board)
At the start: 2 copper layers, 76.2 x 69.9 mm, 35 parts, among them J1 Conn_01x01, J10 Conn_01x02, J11 Conn_01x01, J12 Conn_01x01, J13 Conn_01x01, J14 Conn_01x01, J15 Conn_01x01, J16 Conn_01x01, J2 Conn_01x01, J3 Conn_01x01, J4 Conn_01x01, J5 Conn_01x01, J6 Conn_01x01, J7 Conn_01x02, J8 Conn_01x01, J9 Conn_01x01, U1 TPS3700DDCR, U2 BTS50010-1TAD

Commit message: v1.1
Parts:
- removed the J8 at (111.8, 57.1)
- removed the R4 at (100.3, 55.9)
- added D1: 5.6V, Diode_SMD:D_SOD-123, F.Cu at (91.7, 48.1)
- added J7: Conn_01x03, Connector_PinHeader_2.54mm:PinHeader_1x03_P2.54mm_Vertical, F.Cu at (114.2, 45.7)
- added R5: 0, Resistor_SMD:R_0805_2012Metric_Pad1.20x1.40mm_HandSolder, F.Cu at (97.8, 54.0)
- added R6: 0, Resistor_SMD:R_0805_2012Metric_Pad1.20x1.40mm_HandSolder, F.Cu at (100.5, 54.0)
- added R7: 0, Resistor_SMD:R_0805_2012Metric_Pad1.20x1.40mm_HandSolder, F.Cu at (88.9, 48.3)
- added SW1: SW_Push, Button_Switch_SMD:SW_SPST_PTS810, F.Cu at (114.6, 70.1)
- J9: value Conn_01x01 -> Conn_01x02; footprint Connector_Wire:SolderWire-0.5sqmm_1x01_D0.9mm_OD2.1mm -> Connector_PinHeader_2.54mm:PinHeader_1x02_P2.54mm_Vertical
- moved RV1 28.1 mm to (96.4, 34.3)
- moved R1 13.1 mm to (91.7, 43.3), turned to 90 degrees
- moved RV2 10.8 mm to (106.7, 34.3)
- moved R3 9.17 mm to (108.0, 48.3)
- moved C1 7.75 mm to (98.9, 44.3)
- moved J9 5.97 mm to (114.4, 59.4)
- moved R4 3.18 mm to (95.2, 54.0)
- renumbered C3 to C1, C1 to C2, C2 to C3, J7 to J8, R2 to R1, R1 to R2, R5 to R3, R3 to R4, RV2 to RV1, RV1 to RV2
Connections:
- J9 pad 1: GND -> /EN
- R3 pad 2: Net-(R5-Pad2) -> Net-(R3-Pad2)
- RV2 pad 1: Net-(R5-Pad2) -> GND
- RV2 pad 3: GND -> Net-(R3-Pad2)
- U1 pad 1: /EN -> Net-(U1-Pad1)
- U1 pad 6: /EN -> Net-(U1-Pad6)
- U2 pad 3: /IS -> Net-(U2-Pad3)
Routing:
- net Net-(R5-Pad2): track 23.4 -> 0.00 mm
- net Net-(R3-Pad2): track 0.00 -> 22.7 mm
- net /EN: track 36.1 -> 53.8 mm
- net /IS: track 28.5 -> 11.5 mm, vias 2 -> 0
- net GND: track 16.2 -> 32.7 mm
- net Net-(U2-Pad3): track 0.00 -> 16.5 mm, vias 0 -> 2
- net VDD: track 43.0 -> 59.0 mm
- net /Voff: track 10.7 -> 19.4 mm
- net Net-(R1-Pad2): track 10.3 -> 15.6 mm
- net /Vsense: track 11.2 -> 6.64 mm
- net Net-(U1-Pad1): track 0.00 -> 3.73 mm
- net Net-(U1-Pad6): track 0.00 -> 3.70 mm
Other:
- board text added: "Cutoff v1.1 ch@murgatroid.com (C) 2021"
- board text removed: "Cutoff v1.0 ch@murgatroid.com (C) 2021"
- board text removed: "Vsense"
