File: cutoff/cutoff.kicad_sch (KiCad schematic)
At the start: 31 parts, among them J1 Conn_01x01, J10 Conn_01x01, J11 Conn_01x01, J12 Conn_01x01, J13 Conn_01x01, J14 Conn_01x01, J15 Conn_01x01, J2 Conn_01x01, J3 Conn_01x01, J4 Conn_01x01, J5 Conn_01x01, J6 Conn_01x01, J7 Conn_01x01, J8 Conn_01x01, J9 Conn_01x01, U1 TPS3700DDCR, U2 BTS50010-1TAD

Commit message: .
Parts:
- R5: value R -> 1K
Other:
- title: (none) -> 12V Cutoff
- moved on the sheet: C1, C2, C3, D1, D2, J1, J10, J11, J12, J13, J14, J15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

Commit message: .
Parts:
- removed D1, D2: D_Zener, Diode_SMD:D_1206_3216Metric_Pad1.42x1.75mm_HandSolder, symbol Device:D_Zener
- removed R3, R4: R, Resistor_SMD:R_0805_2012Metric_Pad1.20x1.40mm_HandSolder, symbol Device:R
- added C4: 0.1u, Capacitor_SMD:C_0805_2012Metric_Pad1.18x1.45mm_HandSolder, symbol Device:C
- C1, C2: value C -> 10n
- C3: value C -> 0.1u
- R1: value R -> 2M
- R2: value R -> 1M
- RV1: value 10K -> 100K
- RV2: value 10K -> 5K
- renumbered R5 to R3, R6 to R4
Connections:
- net GND: now also RV1.3, RV2.3, C4.2; no longer R3.2
- net VDD: now also C3.1, C4.1
- net at C1.1, RV1.2, U1.3 (INA+): now also R2.1
- net at R3.1, U2.3 (IS): now also C2.1, U1.4 (INB-); no longer C3.1
- net at RV2.1: now also R3.2, RV2.2
Other:
- moved on the sheet: C1, C2, J1, J10, J11, J12, J13, J14, J15, J2, J3, J4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

Commit message: wip
Parts:
- removed J15: Conn_01x01, Connector_Wire:SolderWire-2.5sqmm_1x01_D2.4mm_OD4.4mm, symbol Connector_Generic:Conn_01x01
- added F1: Fuse, Fuse:Fuseholder_Blade_Mini_Keystone_3568, symbol Device:Fuse
- added H1, H2, H3, H4, H5: MountingHole_Pad, MountingHole:MountingHole_3.2mm_M3_Pad, symbol Mechanical:MountingHole_Pad
- added J16, J17: Conn_01x02, connectors_anderson:45A-VERT-PAIR, symbol Connector_Generic:Conn_01x02
- RV1, RV2: footprint Potentiometer_SMD:Potentiometer_Bourns_3224W_Vertical -> Potentiometer_SMD:Potentiometer_Bourns_3224X_Vertical
Connections:
- net GND: now also H1.1, H2.1, H3.1, H4.1, H5.1, J16.2 (Pin_2), J17.2 (Pin_2)
- net VDD: now also F1.1; no longer J5.1 (Pin_1), J6.1 (Pin_1), J7.1 (Pin_1)
- net Vis: now reaches C2.1, R3.1, U1.4 (INB-), U2.3 (IS)
- net OUT: now reaches J2.1 (Pin_1), J3.1 (Pin_1), J4.1 (Pin_1), U2.5 (OUT), U2.6 (OUT), U2.7 (OUT)
- net OUT: now also J16.1 (Pin_1), J17.1 (Pin_1)
- net Vsense: now reaches J1.1 (Pin_1), JP1.1 (A), R1.1
- net Vcut: now reaches C1.1, R2.1, RV1.2, U1.3 (INA+)
- new net VIN: F1.2, J5.1 (Pin_1), J6.1 (Pin_1), J7.1 (Pin_1)
Other:
- note added: "Place near U1 and U2."

Commit message: wip
Parts:
- removed JP1: SolderJumper_2_Open, Jumper:SolderJumper-2_P1.3mm_Open_Pad1.0x1.5mm, symbol Jumper:SolderJumper_2_Open
- added R5: *0, Resistor_SMD:R_0805_2012Metric_Pad1.20x1.40mm_HandSolder, symbol Device:R
Connections:
- net VDD: now also R5.2
- net Vsense: now also R5.1
- net EN: now reaches R4.2, U1.1 (OUTA), U1.6 (OUTB), U2.2 (IN)
- net Vcut renamed Voff
- net Vis renamed IS
Changed lines of the file:
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@@
     (stroke (width 0) (type solid) (color 0 0 0 0))
   )
-  (wire (pts (xy 133.985 93.345) (xy 142.875 93.345))
+  (wire (pts (xy 133.985 93.345) (xy 138.43 93.345))
     (stroke (width 0) (type solid) (color 0 0 0 0))
   )
   (wire (pts (xy 138.43 93.345) (xy 138.43 117.475))
+    (stroke (width 0) (type solid) (color 0 0 0 0))
+  )
+  (wire (pts (xy 138.43 93.345) (xy 142.875 93.345))
     (stroke (width 0) (type solid) (color 0 0 0 0))
   )
@@
     (effects (font (size 1.27 1.27)) (justify right bottom))
   )
-  (label "Vcut" (at 67.31 90.805 180)
+  (label "Voff" (at 67.31 90.805 180)
     (effects (font (size 1.27 1.27)) (justify right bottom))
   )
-  (label "Vis" (at 67.31 93.345 180)
+  (label "IS" (at 67.31 93.345 180)
+    (effects (font (size 1.27 1.27)) (justify right bottom))
+  )
+  (label "EN" (at 111.125 90.805 180)
     (effects (font (size 1.27 1.27)) (justify right bottom))
   )
@@
     (pin "2")
   )
+  (symbol (lib_id "Device:R") (at 41.275 74.295 90) (unit 1)
+    (in_bom yes) (on_board yes)
+    (property "Reference" "R5" (id 0) (at 41.275 76.835 90)
+      (effects (font (size 1.27 1.27)) (justify left))
+    )
+    (property "Value" "*0" (id 1) (at 43.815 76.835 90)
+      (effects (font (size 1.27 1.27)) (justify left))
+    )
+    (property "Footprint" "Resistor_SMD:R_0805_2012Metric_Pad1.20x1.40mm_HandSolder" (id 2) (at 41.275 76.073 90)
+      (effects (font (size 1.27 1.27)) hide)
+    )
+    (property "Datasheet" "~" (id 3) (at 41.275 74.295 0)
+      (effects (font (size 1.27 1.27)) hide)
+    )
+    (pin "1")
+    (pin "2")
+  )
   (symbol (lib_id "Device:R") (at 113.665 102.235 0) (unit 1)
     (in_bom yes) (on_board yes)
@@
     )
     (pin "1")
-  )
-  (symbol (lib_id "Jumper:SolderJumper_2_Open") (at 41.275 74.295 0) (unit 1)
-    (in_bom yes) (on_board yes)
-    (property "Reference" "JP1" (id 0) (at 41.275 67.945 0))
-    (property "Value" "SolderJumper_2_Open" (id 1) (at 41.275 70.485 0))
-    (property "Footprint" "Jumper:SolderJumper-2_P1.3mm_Open_Pad1.0x1.5mm" (id 2) (at 41.275 74.295 0)
-      (effects (font (size 1.27 1.27)) hide)
-    )
-    (property "Datasheet" "~" (id 3) (at 41.275 74.295 0)
-      (effects (font (size 1.27 1.27)) hide)
-    )
-    (pin "1")
-    (pin "2")
   )
   (symbol (lib_id "Mechanical:MountingHole_Pad") (at 237.49 120.015 0) (unit 1)
@@
       (reference "J17") (unit 1) (value "Conn_01x02") (footprint "connectors_anderson:45A-VERT-PAIR")
     )
-    (path "/a416edeb-eb43-460c-9fd1-c20901e99d91"
-      (reference "JP1") (unit 1) (value "SolderJumper_2_Open") (footprint "Jumper:SolderJumper-2_P1.3mm_Open_Pad1.0x1.5mm")
-    )
     (path "/8b815f9c-7b52-4e54-8794-db6cc3b88ae2"
       (reference "R1") (unit 1) (value "2M") (footprint "Resistor_SMD:R_0805_2012Metric_Pad1.20x1.40mm_HandSolder")
@@
       (reference "R4") (unit 1) (value "20K") (footprint "Resistor_SMD:R_0805_2012Metric_Pad1.20x1.40mm_HandSolder")
     )
+    (path "/ffcb17f9-0800-4ccb-a931-479429b40133"
+      (reference "R5") (unit 1) (value "*0") (footprint "Resistor_SMD:R_0805_2012Metric_Pad1.20x1.40mm_HandSolder")
+    )
     (path "/d5b090bc-f766-46c3-b778-a68417655b2c"

Commit message: wip
Parts:
- J8: renamed from J1; footprint Connector_Wire:SolderWire-2.5sqmm_1x01_D2.4mm_OD4.4mm -> Connector_Wire:SolderWire-0.5sqmm_1x01_D0.9mm_OD2.1mm
- J9: renamed from J13; footprint Connector_Wire:SolderWire-2.5sqmm_1x01_D2.4mm_OD4.4mm -> Connector_Wire:SolderWire-0.5sqmm_1x01_D0.9mm_OD2.1mm
- renumbered C2 to C1, C1 to C2, C4 to C3, C3 to C4, H3 to H1, H5 to H3, H1 to H5, J6 to J1, J16 to J10, J3 to J11, J4 to J12, J2 to J13, J12 to J14, J11 to J15, J9 to J16, J7 to J2, J5 to J3, J8 to J4, J10 to J5, J14 to J6, J17 to J7, R2 to R1, R3 to R2, R4 to R3, R5 to R4, R1 to R5
Other:
- moved on the sheet: J6, J9

Commit message: v1.1
Parts:
- removed J8, J9: Conn_01x01, Connector_Wire:SolderWire-0.5sqmm_1x01_D0.9mm_OD2.1mm, symbol Connector_Generic:Conn_01x01
- removed R4: *0, Resistor_SMD:R_0805_2012Metric_Pad1.20x1.40mm_HandSolder, symbol Device:R
- added D1: 5.6V, Diode_SMD:D_SOD-123, symbol Device:D_Zener
- added J7: Conn_01x03, Connector_PinHeader_2.54mm:PinHeader_1x03_P2.54mm_Vertical, symbol Connector_Generic:Conn_01x03
- added J9: Conn_01x02, Connector_PinHeader_2.54mm:PinHeader_1x02_P2.54mm_Vertical, symbol Connector_Generic:Conn_01x02
- added R5, R6, R7: 0, Resistor_SMD:R_0805_2012Metric_Pad1.20x1.40mm_HandSolder, symbol Device:R
- added SW1: SW_Push, Button_Switch_SMD:SW_SPST_PTS810, symbol Switch:SW_Push
- RV1: renamed from RV2; symbol Device:R_Potentiometer_Trim -> Device:R_POT_TRIM
- RV2: renamed from RV1; symbol Device:R_Potentiometer_Trim -> Device:R_POT_TRIM
- renumbered C3 to C1, C1 to C2, C2 to C3, J7 to J8, R2 to R1, R1 to R2, R5 to R3, R3 to R4
Connections:
- net EN: now also J9.1 (Pin_1), R5.2, R6.2, SW1.2; no longer U1.1 (OUTA), U1.6 (OUTB)
- net GND: now also RV2.1, D1.2 (A), J7.3 (Pin_3), J9.2 (Pin_2), SW1.1; no longer RV2.3
- net IS: now also D1.1 (K), R7.1; no longer U2.3 (IS)
- net VDD: now also J7.1 (Pin_1)
- net Vsense: now also J7.2 (Pin_2)
- net at R3.2: now also RV2.3; no longer RV2.1
- new net: R6.1, U1.1 (OUTA)
- new net: R7.2, U2.3 (IS)
- new net: R5.1, U1.6 (OUTB)
Other:
- note added: "Zener clamp required as fault condition exceeds INB- recommended and max."
- moved on the sheet: C1, C2, C3, C4, F1, H1, H2, H3, H4, H5, J1, J10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
