File: cutoff/cutoff.kicad_sch (KiCad schematic)
At the start: 39 parts, among them J1 Conn_01x01, J10 Conn_01x02, J11 Conn_01x01, J12 Conn_01x01, J13 Conn_01x01, J14 Conn_01x01, J15 Conn_01x01, J16 Conn_01x01, J2 Conn_01x01, J3 Conn_01x01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

Commit message: gnuplot file
Other:
- note added: "INA+ < V_itp_ - V_hys_ => OUTA driven low INB- > V_itp_ => OUTB driver low V_itp_ = 400 mV, V_hys_ = 5.5 mV"
- note added: "V_off_ (min) = 0 V at CCW with V_sense_ dropped over 2M + 100K = 2.1M V_off_ (max) = 0.43 * V_sense_ at CW with V_sense_ dropped over 2M + (100K || 1M) = 2M + 90K"
- note added: "Zener clamp required as fault condition exceeds INB- recommended (6.5V) and max (7V)."
- note removed: "Zener clamp required as fault condition exceeds INB- recommended and max."
